Commit message: Update prebuilt URDF to remove an invalid backtick character.

File: robots/hsrb4s.urdf (robot description, URDF)
Before this commit: robot hsrb, 48 links, 47 joints
Links:
- link hand_l_finger_vacuum_frame: geometry collision box size=0.008 0.008 0.02; visual box size=0.008 0.008 0.02
- link head_l_stereo_camera_link: geometry collision mesh filename=package://hsrb_meshes/meshes/sensors/head_camera.dae; visual mesh filename=package://hsrb_meshes/meshes/sensors/head_camera.dae
- link head_r_stereo_camera_link: geometry collision mesh filename=package://hsrb_meshes/meshes/sensors/head_camera.dae; visual mesh filename=package://hsrb_meshes/meshes/sensors/head_camera.dae
Joints:
- joint base_b_bumper_joint: origin xyz=0.0 0.0013 0.0 rpy=0.0 0.0 3.14159265359 -> xyz=0.0 0.0013 0.0 rpy=0.0 0.0 3.141592653589793
- joint hand_camera_gazebo_frame_joint: origin xyz=0 0 0 rpy=1.57079632679 -1.57079632679 0 -> xyz=0 0 0 rpy=1.5707963267948966 -1.5707963267948966 0
- joint hand_l_finger_tip_frame_joint: origin xyz=0.01675 0.01865 0.04289 rpy=-1.57079632679 0.0 0.0 -> xyz=0.01675 0.01865 0.04289 rpy=-1.5707963267948966 0.0 0.0
- joint hand_l_finger_vacuum_frame_joint: origin xyz=0.00475 -0.011539 0.03322 rpy=0.785398163397 0.0 0.0 -> xyz=0.00475 -0.011539 0.03322 rpy=0.7853981633974483 0.0 0.0
- joint hand_palm_joint: origin xyz=0.012 0.0 0.1405 rpy=0.0 0.0 3.14159265359 -> xyz=0.012 0.0 0.1405 rpy=0.0 0.0 3.141592653589793
- joint hand_r_finger_tip_frame_joint: origin xyz=0.01675 -0.01865 0.04289 rpy=1.57079632679 0.0 0.0 -> xyz=0.01675 -0.01865 0.04289 rpy=1.5707963267948966 0.0 0.0
- joint head_center_camera_frame_joint: origin xyz=0.0195 0.0 0.061 rpy=-1.57079632679 0.0 -1.57079632679 -> xyz=0.0195 0.0 0.061 rpy=-1.5707963267948966 0.0 -1.5707963267948966
- joint head_center_camera_gazebo_frame_joint: origin xyz=0 0 0 rpy=1.57079632679 -1.57079632679 0.0 -> xyz=0 0 0 rpy=1.5707963267948966 -1.5707963267948966 0.0
- joint head_l_stereo_camera_gazebo_frame_joint: origin xyz=0 0 0 rpy=1.57079632679 -1.57079632679 0.0 -> xyz=0 0 0 rpy=1.5707963267948966 -1.5707963267948966 0.0
- joint head_l_stereo_camera_joint: origin xyz=0.02 0.07 0.061 rpy=-1.57079632679 0.0 -1.57079632679 -> xyz=0.02 0.07 0.061 rpy=-1.5707963267948966 0.0 -1.5707963267948966
- joint head_r_stereo_camera_gazebo_frame_joint: origin xyz=0 0 0 rpy=1.57079632679 -1.57079632679 0.0 -> xyz=0 0 0 rpy=1.5707963267948966 -1.5707963267948966 0.0
- joint head_r_stereo_camera_joint: origin xyz=0.02 -0.07 0.061 rpy=-1.57079632679 0.0 -1.57079632679 -> xyz=0.02 -0.07 0.061 rpy=-1.5707963267948966 0.0 -1.5707963267948966
- joint head_rgbd_sensor_gazebo_frame_joint: origin xyz=0 0 0 rpy=1.57079632679 -1.57079632679 0.0 -> xyz=0 0 0 rpy=1.5707963267948966 -1.5707963267948966 0.0
- joint head_rgbd_sensor_joint: origin xyz=-0.079796 0.022 0.215172 rpy=-1.57079632679 0.0 -1.57079632679 -> xyz=-0.079796 0.022 0.215172 rpy=-1.5707963267948966 0.0 -1.5707963267948966
- joint wrist_ft_sensor_frame_inverse_joint: origin xyz=0.0 0.0 0.0735 rpy=-3.14159265359 0.0 0.0 -> xyz=0.0 0.0 0.0735 rpy=-3.141592653589793 0.0 0.0
- joint wrist_ft_sensor_frame_joint: origin xyz=0.0 0.0 0.0735 rpy=3.14159265359 0.0 0.0 -> xyz=0.0 0.0 0.0735 rpy=3.141592653589793 0.0 0.0
